File: MCU Datalogger.kicad_sch (KiCad schematic)
At the start: 25 parts, among them U1 24LC1025, U2 DS1337S+, U3 24LC1025, U4 ATMEGA328-AU, Y1 32.768 KHz, Y2 16 MHz

Commit message: Complete with adding comments in the sheet.
Other:
- note added: "EEPROM"
- note added: "MCU"
- note added: "Mounting"
- note added: "RTC clock"
- moved on the sheet: C1, R2, R3, U2, Y1
